Commit message: Removed most absolute paths to files, fixed bugs

File: robot_description/sensors/urdf/hokuyo3d.urdf.xacro (robot description, xacro)
@@ -17,5 +17,5 @@
 			<origin xyz="0 0 0" rpy="0 0 0"/>
 			<geometry>
-	     		<mesh filename="file:///home/patrik/catkin_ws/src/mech_ros/robot_description/sensors/meshes/hokuyo3d.stl"/>
+	     		<mesh filename="$(find mech_ros)/robot_description/sensors/meshes/hokuyo3d.stl"/>
 			</geometry>
 		</visual>

File: robot_description/sensors/urdf/hokuyo_urg04lx.urdf.xacro (robot description, xacro)
@@ -34,5 +34,5 @@
         <origin xyz="0 0 -0.05" rpy="0 0 0"/>
         <geometry>
-            <mesh filename="file:///home/patrik/catkin_ws/src/mech_ros/robot_description/sensors/meshes/hokuyo_urg_04lx.dae"/>
+            <mesh filename="$(find mech_ros)/robot_description/sensors/meshes/hokuyo_urg_04lx.dae"/>
         </geometry>
       </visual>

File: robot_description/sensors/urdf/hokuyo_ust10lx.urdf.xacro (robot description, xacro)
@@ -43,5 +43,5 @@
         <origin xyz="0 0 0.0" rpy="0 0 0"/>
         <geometry>
-            <mesh filename="file:///home/patrik/catkin_ws/src/mech_ros/robot_description/sensors/meshes/hokuyo_ust_10lx.dae"/>
+            <mesh filename="$(find mech_ros)/robot_description/sensors/meshes/hokuyo_ust_10lx.dae"/>
         </geometry>
       </visual>

File: robot_description/sensors/urdf/pi_camera.urdf.xacro (robot description, xacro)
@@ -33,5 +33,5 @@
 	<origin xyz="0 0 0" rpy="0 ${-PI/2} ${PI}"/>
      <geometry>
-        <mesh filename="file:///home/patrik/catkin_ws/src/mech_ros/robot_description/meshes/Camera_2000_simplified.stl" scale="${Scale}"/>
+        <mesh filename="$(find mech_ros)/robot_description/meshes/Camera_2000_simplified.stl" scale="${Scale}"/>
       </geometry>
      <material name="camera_color"/>

File: robot_description/urdf/mechROS.xacro (robot description, xacro)
@@ -37,13 +37,9 @@
    <color rgba=".01 1 .5 1"/>
 </material>
-<!--<material name="tire_texture">-->
-<!--    <texture filename="package://robot_description/textures/rubber.jpg" />-->
-<!--</material>-->
 <!-- Import files -->
-	<!--	<xacro:include filename="package://robot_description/urdf/rubber_wheel.urdf.xacro"/>-->
-	<xacro:include filename="/home/patrik/catkin_ws/src/mech_ros/robot_description/urdf/rubber_wheel.urdf.xacro"/>
-	<xacro:include filename="/home/patrik/catkin_ws/src/mech_ros/robot_description/urdf/mechROS_control.gazebo.xacro"/>
-	<!--<xacro:include filename="file:///home/patrik/catkin_ws/src/mech_ros/robot_description/sensors/urdf/all_sensors.urdf.xacro" />-->
-	<xacro:include filename="/home/patrik/catkin_ws/src/mech_ros/robot_description/sensors/urdf/all_sensors.urdf.xacro" />
+	<xacro:include filename="$(find mech_ros)/robot_description/urdf/rubber_wheel.urdf.xacro"/>
+	<xacro:include filename="$(find mech_ros)/robot_description/urdf/mechROS_control.gazebo.xacro"/>
+	<xacro:include filename="$(find mech_ros)/robot_description/urdf/mechROS_control.gazebo.xacro"/>
+	<xacro:include filename="$(find mech_ros)/robot_description/sensors/urdf/all_sensors.urdf.xacro" />
 <xacro:property name="PI" value="3.1415926535897931"/>
 <material name="gray_color">
@@ -56,6 +52,5 @@
      <origin xyz="0.011 -0.060276 0" rpy="${PI/2} 0 ${PI/2}"/>
      <geometry>
-<!--        <mesh filename="package://robot_description/meshes/Chassis.stl"/>-->
-	<mesh filename="file:///home/patrik/catkin_ws/src/mech_ros/robot_description/meshes/Chassis_10000.stl" scale="${Scale}"/>
+			<mesh filename="$(find mech_ros)/robot_description/meshes/Chassis_10000.stl" scale="${Scale}"/>
 <!--	<cylinder length="0.2" radius="0.4" />-->
      </geometry>
@@ -117,27 +112,4 @@
 		<origin xyz="0.0 0.0 0.0804" rpy="0 0 0"/>
 	</xacro:sensor_hokuyo_urg04lx>
-<!-- Import Laser -->
-	 <!-- <xacro:sensor_hokuyo_ust10lx prefix="laser" parent="$(arg prefix)base_link">
-	<origin xyz="0.00 0 0.0804" rpy="0 0 0"/>
-	</xacro:sensor_hokuyo_ust10lx>  -->
 <xacro:ros_control/>
-<!-- <xacro:skid_steering broadcastOdomTF="false" prefix="$(arg prefix)" wheelSeparation="0.18" wheelDiameter="0.1"/> -->
-<!--<link name="camera">-->
-<!--    <visual>-->
-<!--	<origin xyz="0 0 0" rpy="0 ${-PI/2} ${PI}"/>-->
-<!--     <geometry>-->
-<!--        <mesh filename="file:///home/patrik/catkin_ws/src/mech_ros/robot_description/meshes/Camera.stl" scale="${Scale}"/>-->
-<!--      </geometry>-->
-<!--     <material name="camera_color"/>-->
-<!--    </visual>-->
-<!--    <collision>-->
-<!--      <origin xyz="0 0 0" rpy="0 0 0"/>-->
-<!--      <geometry>-->
-<!--        <box size="0.01 0.2 0.05"/>-->
-<!--      </geometry>-->
-<!--    </collision>-->
-<!--</link>-->
-<!-- JOINTS -->
-<!-- ////////////////////////////////////////////////// -->
-<!--<xacro:Joint_f name="Body" parent="base_link" child="camera" xyz="0.088 0 0.0204" rpy="0 0 0"/>-->
 </robot>

File: robot_description/urdf/mechROS_control.gazebo.xacro (robot description, xacro)
@@ -33,34 +33,3 @@
     </gazebo>
   </xacro:macro>
-<!--  -->
-<!--  <xacro:macro name="omni_steering" params="prefix publish_tf">-->
-<!--		<gazebo>-->
-<!--	    <plugin name="omni_steering" filename="libgazebo_ros_planar_move.so">-->
-<!--	      <commandTopic>robotnik_base_control/cmd_vel</commandTopic>  -->
-<!--	      <odometryTopic>robotnik_base_control/odom</odometryTopic>-->
-<!--	      <odometryFrame>${prefix}odom</odometryFrame>-->
-<!--	      <odometryRate>50.0</odometryRate>-->
-<!--	      <robotBaseFrame>${prefix}base_footprint</robotBaseFrame>-->
-<!--	      <publishTF>${publish_tf}</publishTF>-->
-<!--	    </plugin>-->
-<!--	  </gazebo>-->
-<!--  </xacro:macro>-->
-<!--  <xacro:macro name="ros_force_based_move" params="publish_tf prefix">-->
-<!--	  <gazebo>-->
-<!--		 <plugin name="ros_force_based_move" filename="libgazebo_ros_force_based_move.so">-->
-<!--			 <commandTopic>robotnik_base_control/cmd_vel</commandTopic>  -->
-<!--			 <odometryTopic>robotnik_base_control/odom</odometryTopic>-->
-<!--	         <odometryFrame>${prefix}odom</odometryFrame>-->
-<!--			 <yaw_velocity_p_gain>10000.0</yaw_velocity_p_gain>-->
-<!--			 <x_velocity_p_gain>10000.0</x_velocity_p_gain>-->
-<!--			 <y_velocity_p_gain>10000.0</y_velocity_p_gain>-->
-<!--			 <robotBaseFrame>${prefix}base_footprint</robotBaseFrame>-->
-<!--			 <odometryRate>50.0</odometryRate>-->
-<!--			 <publishOdometryTf>${publish_tf}</publishOdometryTf>-->
-<!--		 </plugin>-->
-<!--	  </gazebo>-->
-<!--  </xacro:macro>-->
-<!--  <gazebo reference="base_footprint">-->
-<!--    <material>Gazebo/Green</material>-->
-<!--  </gazebo>-->
 </robot>

File: robot_description/urdf/rubber_wheel.urdf.xacro (robot description, xacro)
@@ -29,5 +29,5 @@
 <xacro:property name="Scale" value="${scale} ${scale} ${scale}"/>
 <material name="tire_texture">
-    <texture filename="file:///home/patrik/catkin_ws/src/mech_ros/robot_description/textures/rubber.jpg" />
+    <texture filename="$(find mech_ros)/robot_description/textures/rubber.jpg" />
 </material>
   <xacro:macro name="rubber_wheel" params="prefix parent *origin reflect">
@@ -38,5 +38,4 @@
       <xacro:insert_block name="origin" />
       <axis xyz="0 1 0" rpy="0 0 0" />
-      <!-- <limit effort="100" velocity="100"/> -->
       <limit effort="1000" velocity="1000" />
       <joint_properties damping="0.0" friction="0.0"/>
@@ -51,5 +50,5 @@
 	      </xacro:unless>
         <geometry>
-             <mesh filename="file:///home/patrik/catkin_ws/src/mech_ros/robot_description/meshes/Wheel_hub_simplified.stl" scale="${Scale}"/>
+             <mesh filename="$(find mech_ros)/robot_description/meshes/Wheel_hub_simplified.stl" scale="${Scale}"/>
         </geometry>
 	      <material name="tire_texture"/>
@@ -69,10 +68,4 @@
         <friction>
           <ode>
-          <!-- This works well enough -->
-            <!-- <mu>1.0</mu>
-            <mu2>0.3</mu2>
-            <slip1>0.5</slip1>
-            <slip2>0.0</slip2>
-            <fdir1 value="1 0 0"/> -->
             <mu>1.0</mu>
             <mu2>1.0</mu2>
@@ -109,23 +102,5 @@
       </actuator>
     </transmission>
-	<!-- <transmission name="${prefix}_wheel_joint_trans">
-      <type>transmission_interface/SimpleTransmission</type>
-      <joint name="${prefix}_wheel_joint">
-        <hardwareInterface>hardware_interface/EffortJointInterface</hardwareInterface>
-      </joint>
-      <actuator name="${prefix}_wheel_joint_motor">
-        <mechanicalReduction>1</mechanicalReduction>
-        <hardwareInterface>hardware_interface/EffortJointInterface</hardwareInterface>
-      </actuator>
-  </transmission> -->
     <gazebo reference="${prefix}_wheel">
-			<!-- <mu1 value="1.0"/>
-      <mu2 value="1.0"/>
-			<kp value="10000000.0" />
-			<kd value="1.0" />
-			<fdir1 value="1 0 0"/> -->
-			<!-- <mu2 value="1.0"/> -->
-			<!-- <slip11 value="0.5"/>
-			<slip2 value="0.0"/>       -->
 	    <material>Gazebo/Residential</material>
       <turnGravityOff>false</turnGravityOff>
