Commit message: Modified paths to filename

File: robot_description/sensors/urdf/hokuyo_urg04lx.urdf.xacro (robot description, xacro)
@@ -1,4 +1,5 @@
 <?xml version="1.0"?>
-<robot name="sensor_hokuyo_urg04lx" xmlns:xacro="http://www.ros.org/wiki/xacro">
+<robot name="sensor_hokuyo_urg04lx"
+  xmlns:xacro="http://www.ros.org/wiki/xacro">
   <!-- Copyright (c) 2014, Robotnik Automation
 All rights reserved.
@@ -34,5 +35,5 @@
         <origin xyz="0 0 -0.05" rpy="0 0 0"/>
         <geometry>
-            <mesh filename="$(find mech_ros)/robot_description/sensors/meshes/hokuyo_urg_04lx.dae"/>
+          <mesh filename="package://mech_ros/robot_description/sensors/meshes/hokuyo_urg_04lx.dae"/>
         </geometry>
       </visual>
@@ -44,10 +45,10 @@
     </link>
     <link name="${prefix}_link">
-	</link>
+    </link>
     <joint name="${prefix}_joint" type="fixed">
       <parent link="${prefix}_base_link"/>
       <child link="${prefix}_link"/>
       <origin xyz="0.0 0.0 0.0" rpy="0 0 0"/>
-	</joint>
+    </joint>
     <!-- Hokuyo sensor for simulation -->
     <sensor_hokuyo_urg04lx_gazebo/>
@@ -55,35 +56,35 @@
   <xacro:macro name="sensor_hokuyo_urg04lx_gazebo">
     <gazebo reference="${prefix}_link">
-			<sensor type="ray" name="${prefix}_sensor">
-				<pose>0 0 0 0 0 0</pose>
-				<visualize>false</visualize>
-				<update_rate>10</update_rate>
-				<ray>
-					<scan>
-						<horizontal>
-							<samples>640</samples>
-							<resolution>1</resolution>
-							<min_angle>${min_angle}</min_angle>
-							<max_angle>${max_angle}</max_angle>
-						</horizontal>
-					</scan>
-					<range>
-						<min>0.08</min>
-						<max>4.0</max>
-						<resolution>0.00628318531</resolution>
-					</range>
-					<noise>
-						<type>gaussian</type>
-						<mean>0.0</mean>
-						<stddev>0.01</stddev>
-					</noise>
-				</ray>
-				<plugin name="${prefix}_controller" filename="libgazebo_ros_laser.so">
-					<topicName>${prefix_topic}/scan</topicName>
-					<frameName>${prefix}_link</frameName>
-					<ignoreTfPrefix>1</ignoreTfPrefix>
-				</plugin>
-			</sensor>
-	</gazebo>
+      <sensor type="ray" name="${prefix}_sensor">
+        <pose>0 0 0 0 0 0</pose>
+        <visualize>false</visualize>
+        <update_rate>10</update_rate>
+        <ray>
+          <scan>
+            <horizontal>
+              <samples>640</samples>
+              <resolution>1</resolution>
+              <min_angle>${min_angle}</min_angle>
+              <max_angle>${max_angle}</max_angle>
+            </horizontal>
+          </scan>
+          <range>
+            <min>0.08</min>
+            <max>4.0</max>
+            <resolution>0.00628318531</resolution>
+          </range>
+          <noise>
+            <type>gaussian</type>
+            <mean>0.0</mean>
+            <stddev>0.01</stddev>
+          </noise>
+        </ray>
+        <plugin name="${prefix}_controller" filename="libgazebo_ros_laser.so">
+          <topicName>${prefix_topic}/scan</topicName>
+          <frameName>${prefix}_link</frameName>
+          <ignoreTfPrefix>1</ignoreTfPrefix>
+        </plugin>
+      </sensor>
+    </gazebo>
   </xacro:macro>
 </robot>

File: robot_description/sensors/urdf/hokuyo_ust10lx.urdf.xacro (robot description, xacro)
@@ -1,5 +1,6 @@
 <?xml version="1.0"?>
-<robot name="sensor_hokuyo_ust10lx" xmlns:xacro="http://www.ros.org/wiki/xacro">
-<!-- Copyright (c) 2014, Robotnik Automation
+<robot name="sensor_hokuyo_ust10lx"
+  xmlns:xacro="http://www.ros.org/wiki/xacro">
+  <!-- Copyright (c) 2014, Robotnik Automation
 All rights reserved.
 Redistribution and use in source and binary forms, with or without
@@ -22,10 +23,10 @@
   <xacro:macro name="sensor_hokuyo_ust10lx" params="prefix parent prefix_topic:='front_laser' *origin min_angle:=-2.3562 max_angle:=2.3562">
     <link name="${prefix}_link">
-	</link>
+    </link>
     <joint name="${prefix}_joint" type="fixed">
       <parent link="${parent}"/>
       <child link="${prefix}_link"/>
       <xacro:insert_block name="origin" />
-	</joint>
+    </joint>
     <joint name="${prefix}_base_joint" type="fixed">
       <origin xyz="0.00 0 -0.05" rpy="0 0 0"/>
@@ -43,5 +44,5 @@
         <origin xyz="0 0 0.0" rpy="0 0 0"/>
         <geometry>
-            <mesh filename="$(find mech_ros)/robot_description/sensors/meshes/hokuyo_ust_10lx.dae"/>
+          <mesh filename="package://mech_ros/robot_description/sensors/meshes/hokuyo_ust_10lx.dae"/>
         </geometry>
       </visual>
@@ -53,36 +54,36 @@
     </link>
     <gazebo reference="${prefix}_link">
-			<sensor type="gpu_ray" name="${prefix}_sensor">
-				<pose>0 0 0 0 0 0</pose>
-				<visualize>false</visualize>
-				<update_rate>40</update_rate>
-				<ray>
-					<scan>
-						<horizontal>
-							<samples>1081</samples>
-							<resolution>1</resolution>
-							<min_angle>${min_angle}</min_angle>
-							<max_angle>${max_angle}</max_angle>
-						</horizontal>
-					</scan>
-					<range>
-						<min>0.06</min>
-						<max>10.0</max>
-						<!-- resolution>0.004363323</resolution -->
-						<resolution>0.004359297</resolution>
-						<!-- resolution>0.001</resolution -->
-					</range>
-					<noise>
-						<type>gaussian</type>
-						<mean>0.0</mean>
-						<stddev>0.01</stddev>
-					</noise>
-				</ray>
-				<plugin name="${prefix}_controller" filename="libgazebo_ros_gpu_laser.so">
-					<topicName>${prefix_topic}/scan</topicName>
-					<frameName>/${prefix}_link</frameName>
-				</plugin>
-			</sensor>
-	</gazebo>
+      <sensor type="gpu_ray" name="${prefix}_sensor">
+        <pose>0 0 0 0 0 0</pose>
+        <visualize>false</visualize>
+        <update_rate>40</update_rate>
+        <ray>
+          <scan>
+            <horizontal>
+              <samples>1081</samples>
+              <resolution>1</resolution>
+              <min_angle>${min_angle}</min_angle>
+              <max_angle>${max_angle}</max_angle>
+            </horizontal>
+          </scan>
+          <range>
+            <min>0.06</min>
+            <max>10.0</max>
+            <!-- resolution>0.004363323</resolution -->
+            <resolution>0.004359297</resolution>
+            <!-- resolution>0.001</resolution -->
+          </range>
+          <noise>
+            <type>gaussian</type>
+            <mean>0.0</mean>
+            <stddev>0.01</stddev>
+          </noise>
+        </ray>
+        <plugin name="${prefix}_controller" filename="libgazebo_ros_gpu_laser.so">
+          <topicName>${prefix_topic}/scan</topicName>
+          <frameName>/${prefix}_link</frameName>
+        </plugin>
+      </sensor>
+    </gazebo>
   </xacro:macro>
 </robot>

File: robot_description/sensors/urdf/pi_camera.urdf.xacro (robot description, xacro)
@@ -1,23 +1,24 @@
 <?xml version="1.0"?>
-<robot name="pi_camera" xmlns:xacro="http://www.ros.org/wiki/xacro">
-<!--Copyright (c) 2014, Robotnik Automation-->
-<!--All rights reserved.-->
-<!--Redistribution and use in source and binary forms, with or without-->
-<!--modification, are permitted provided that the following conditions are met:-->
-<!--* Redistributions of source code must retain the above copyright notice, this-->
-<!--  list of conditions and the following disclaimer.-->
-<!--* Redistributions in binary form must reproduce the above copyright notice,-->
-<!--  this list of conditions and the following disclaimer in the documentation-->
-<!--  and/or other materials provided with the distribution.-->
-<!--THIS SOFTWARE IS PROVIDED BY THE COPYRIGHT HOLDERS AND CONTRIBUTORS "AS IS"-->
-<!--AND ANY EXPRESS OR IMPLIED WARRANTIES, INCLUDING, BUT NOT LIMITED TO, THE-->
-<!--IMPLIED WARRANTIES OF MERCHANTABILITY AND FITNESS FOR A PARTICULAR PURPOSE ARE-->
-<!--DISCLAIMED. IN NO EVENT SHALL THE COPYRIGHT HOLDER OR CONTRIBUTORS BE LIABLE-->
-<!--FOR ANY DIRECT, INDIRECT, INCIDENTAL, SPECIAL, EXEMPLARY, OR CONSEQUENTIAL-->
-<!--DAMAGES (INCLUDING, BUT NOT LIMITED TO, PROCUREMENT OF SUBSTITUTE GOODS OR-->
-<!--SERVICES; LOSS OF USE, DATA, OR PROFITS; OR BUSINESS INTERRUPTION) HOWEVER-->
-<!--CAUSED AND ON ANY THEORY OF LIABILITY, WHETHER IN CONTRACT, STRICT LIABILITY,-->
-<!--OR TORT (INCLUDING NEGLIGENCE OR OTHERWISE) ARISING IN ANY WAY OUT OF THE USE-->
-<!--OF THIS SOFTWARE, EVEN IF ADVISED OF THE POSSIBILITY OF SUCH DAMAGE.-->
+<robot name="pi_camera"
+  xmlns:xacro="http://www.ros.org/wiki/xacro">
+  <!--Copyright (c) 2014, Robotnik Automation-->
+  <!--All rights reserved.-->
+  <!--Redistribution and use in source and binary forms, with or without-->
+  <!--modification, are permitted provided that the following conditions are met:-->
+  <!--* Redistributions of source code must retain the above copyright notice, this-->
+  <!--  list of conditions and the following disclaimer.-->
+  <!--* Redistributions in binary form must reproduce the above copyright notice,-->
+  <!--  this list of conditions and the following disclaimer in the documentation-->
+  <!--  and/or other materials provided with the distribution.-->
+  <!--THIS SOFTWARE IS PROVIDED BY THE COPYRIGHT HOLDERS AND CONTRIBUTORS "AS IS"-->
+  <!--AND ANY EXPRESS OR IMPLIED WARRANTIES, INCLUDING, BUT NOT LIMITED TO, THE-->
+  <!--IMPLIED WARRANTIES OF MERCHANTABILITY AND FITNESS FOR A PARTICULAR PURPOSE ARE-->
+  <!--DISCLAIMED. IN NO EVENT SHALL THE COPYRIGHT HOLDER OR CONTRIBUTORS BE LIABLE-->
+  <!--FOR ANY DIRECT, INDIRECT, INCIDENTAL, SPECIAL, EXEMPLARY, OR CONSEQUENTIAL-->
+  <!--DAMAGES (INCLUDING, BUT NOT LIMITED TO, PROCUREMENT OF SUBSTITUTE GOODS OR-->
+  <!--SERVICES; LOSS OF USE, DATA, OR PROFITS; OR BUSINESS INTERRUPTION) HOWEVER-->
+  <!--CAUSED AND ON ANY THEORY OF LIABILITY, WHETHER IN CONTRACT, STRICT LIABILITY,-->
+  <!--OR TORT (INCLUDING NEGLIGENCE OR OTHERWISE) ARISING IN ANY WAY OUT OF THE USE-->
+  <!--OF THIS SOFTWARE, EVEN IF ADVISED OF THE POSSIBILITY OF SUCH DAMAGE.-->
   <xacro:property name="M_PI" value="3.1415926535897931" />
   <xacro:macro name="pi_camera_sensor" params="prefix parent *origin">
@@ -29,16 +30,16 @@
     </joint>
     <link name="${prefix}_camera_link">
- 	<visual>
-<!--     <origin xyz="0 0 0" rpy="0 ${PI/2} 0"/>-->
-	<origin xyz="0 0 0" rpy="0 ${-PI/2} ${PI}"/>
-     <geometry>
-        <mesh filename="$(find mech_ros)/robot_description/meshes/Camera_2000_simplified.stl" scale="${Scale}"/>
-      </geometry>
-     <material name="camera_color"/>
-    </visual>
+      <visual>
+        <!--     <origin xyz="0 0 0" rpy="0 ${PI/2} 0"/>-->
+        <origin xyz="0 0 0" rpy="0 ${-PI/2} ${PI}"/>
+        <geometry>
+          <mesh filename="package://mech_ros/robot_description/meshes/Camera_2000_simplified.stl" scale="${Scale}"/>
+        </geometry>
+        <material name="camera_color"/>
+      </visual>
       <collision>
         <origin xyz="0.0 0.0 0.0" rpy="0 0 0"/>
         <geometry>
-        <box size="0.001 0.03 0.03"/>
+          <box size="0.001 0.03 0.03"/>
         </geometry>
       </collision>
@@ -50,55 +51,55 @@
       </inertial>
     </link>
-  <!-- camera -->
-  <gazebo reference="${prefix}_camera_link">
-    <sensor type="camera" name="camera1">
-      <update_rate>30.0</update_rate>
-      <camera name="head">
-        <horizontal_fov>1.3962634</horizontal_fov>
-        <image>
-          <width>1280</width>
-          <height>720</height>
-          <format>R8G8B8</format>
-        </image>
-        <clip>
-          <near>0.02</near>
-          <far>300</far>
-        </clip>
-        <noise>
-          <type>gaussian</type>
-          <!-- Noise is sampled independently per pixel on each frame.
+    <!-- camera -->
+    <gazebo reference="${prefix}_camera_link">
+      <sensor type="camera" name="camera1">
+        <update_rate>30.0</update_rate>
+        <camera name="head">
+          <horizontal_fov>1.3962634</horizontal_fov>
+          <image>
+            <width>1280</width>
+            <height>720</height>
+            <format>R8G8B8</format>
+          </image>
+          <clip>
+            <near>0.02</near>
+            <far>300</far>
+          </clip>
+          <noise>
+            <type>gaussian</type>
+            <!-- Noise is sampled independently per pixel on each frame.
                That pixel's noise value is added to each of its color
                channels, which at that point lie in the range [0,1]. -->
-          <mean>0.0</mean>
-          <stddev>0.007</stddev>
-        </noise>
-      </camera>
-      <plugin name="camera_controller" filename="libgazebo_ros_camera.so">
-        <alwaysOn>true</alwaysOn>
-        <updateRate>0.0</updateRate>
-        <cameraName>pi_camera</cameraName>
-        <imageTopicName>image_raw</imageTopicName>
-        <cameraInfoTopicName>camera_info</cameraInfoTopicName>
-        <frameName>front_camera_link</frameName>
-        <hackBaseline>0.0</hackBaseline>
-        <!-- <distortionK1>0.12229709180689073</distortionK1>
+            <mean>0.0</mean>
+            <stddev>0.007</stddev>
+          </noise>
+        </camera>
+        <plugin name="camera_controller" filename="libgazebo_ros_camera.so">
+          <alwaysOn>true</alwaysOn>
+          <updateRate>0.0</updateRate>
+          <cameraName>pi_camera</cameraName>
+          <imageTopicName>image_raw</imageTopicName>
+          <cameraInfoTopicName>camera_info</cameraInfoTopicName>
+          <frameName>front_camera_link</frameName>
+          <hackBaseline>0.0</hackBaseline>
+          <!-- <distortionK1>0.12229709180689073</distortionK1>
         <distortionK2>0.024010173426467347</distortionK2>
         <distortionK3>-1.8227973245663944</distortionK3>
         <distortionT1>0.017489177150311525</distortionT1>
         <distortionT2>0.0025341869220518796</distortionT2> -->
-        <distortionK1>0.0</distortionK1>
-        <distortionK2>0.0</distortionK2>
-        <distortionK3>0.0</distortionK3>
-        <distortionT1>0.0</distortionT1>
-        <distortionT2>0.0</distortionT2>
-        <!-- Added 16.1.2019, if not working due to change, delete -->
-        <!-- <CxPrime>0</CxPrime> -->
-        <!-- <Cx>0.0</Cx>
+          <distortionK1>0.0</distortionK1>
+          <distortionK2>0.0</distortionK2>
+          <distortionK3>0.0</distortionK3>
+          <distortionT1>0.0</distortionT1>
+          <distortionT2>0.0</distortionT2>
+          <!-- Added 16.1.2019, if not working due to change, delete -->
+          <!-- <CxPrime>0</CxPrime> -->
+          <!-- <Cx>0.0</Cx>
         <Cy>0.0</Cy> -->
-        <!-- <focalLength>762.724934</focalLength> -->
-      </plugin>
-    </sensor>
-    <material>Gazebo/Grass</material>
-  </gazebo>
+          <!-- <focalLength>762.724934</focalLength> -->
+        </plugin>
+      </sensor>
+      <material>Gazebo/Grass</material>
+    </gazebo>
   </xacro:macro>
 </robot>

File: robot_description/urdf/mechROS.xacro (robot description, xacro)
@@ -1,5 +1,6 @@
 ﻿<?xml version="1.0"?>
-<robot name="mechROS" xmlns:xacro="http://www.ros.org/wiki/xacro">
-<!-- Copyright (c) 2014, Robotnik Automation
+<robot name="mechROS"
+	xmlns:xacro="http://www.ros.org/wiki/xacro">
+	<!-- Copyright (c) 2014, Robotnik Automation
 All rights reserved.
 Redistribution and use in source and binary forms, with or without
@@ -20,71 +21,72 @@
 OR TORT (INCLUDING NEGLIGENCE OR OTHERWISE) ARISING IN ANY WAY OUT OF THE USE
 OF THIS SOFTWARE, EVEN IF ADVISED OF THE POSSIBILITY OF SUCH DAMAGE. -->
-<!-- PROPERTIES & MACROS -->
-<!-- ////////////////////////////////////////////////// -->
-<!-- Robot name -->
-<xacro:arg name="prefix" default="mechROS_"/>
-<xacro:arg name="wheel_offset_y" default="0.0735" />
-<!-- SCALE definition -->
-<xacro:property name="scale" value="0.01"/>    <!-- meritko-->
-<xacro:property name="Scale" value="${scale} ${scale} ${scale}"/>
-<!-- Wheel parameters -->
-<xacro:property name="wheel_offset_x" value="0.063" />    <!-- x,y,z in translation from base_link to the center of the wheel -->
-<xacro:property name="wheel_offset_y" value="0.0735" />
-<xacro:property name="wheel_offset_z" value="0.018" />
-<!-- MATERIALS -->
-<!-- ////////////////////////////////////////////////// -->
-<material name="camera_color">
-   <color rgba=".01 1 .5 1"/>
-</material>
-<!-- Import files -->
+	<!-- PROPERTIES & MACROS -->
+	<!-- ////////////////////////////////////////////////// -->
+	<!-- Robot name -->
+	<xacro:arg name="prefix" default="mechROS_"/>
+	<xacro:arg name="wheel_offset_y" default="0.0735" />
+	<!-- SCALE definition -->
+	<xacro:property name="scale" value="0.01"/>
+	<!-- meritko-->
+	<xacro:property name="Scale" value="${scale} ${scale} ${scale}"/>
+	<!-- Wheel parameters -->
+	<xacro:property name="wheel_offset_x" value="0.063" />
+	<!-- x,y,z in translation from base_link to the center of the wheel -->
+	<xacro:property name="wheel_offset_y" value="0.0735" />
+	<xacro:property name="wheel_offset_z" value="0.018" />
+	<!-- MATERIALS -->
+	<!-- ////////////////////////////////////////////////// -->
+	<material name="camera_color">
+		<color rgba=".01 1 .5 1"/>
+	</material>
+	<!-- Import files -->
 	<xacro:include filename="$(find mech_ros)/robot_description/urdf/rubber_wheel.urdf.xacro"/>
 	<xacro:include filename="$(find mech_ros)/robot_description/urdf/mechROS_control.gazebo.xacro"/>
 	<xacro:include filename="$(find mech_ros)/robot_description/urdf/mechROS_control.gazebo.xacro"/>
 	<xacro:include filename="$(find mech_ros)/robot_description/sensors/urdf/all_sensors.urdf.xacro" />
-<xacro:property name="PI" value="3.1415926535897931"/>
-<material name="gray_color">
-    <color rgba=".75 .75 .75 1"/>
- </material>
-<!-- LINKS -->
-<!-- ////////////////////////////////////////////////// -->
-<link name="$(arg prefix)base_link">
-    <visual>
-     <origin xyz="0.011 -0.060276 0" rpy="${PI/2} 0 ${PI/2}"/>
-     <geometry>
-			<mesh filename="$(find mech_ros)/robot_description/meshes/Chassis_10000.stl" scale="${Scale}"/>
-<!--	<cylinder length="0.2" radius="0.4" />-->
-     </geometry>
-     <material name="gray_color"/>
-    </visual>
-    <collision>
-      <origin xyz="0.008 0 0.023" rpy="0 0 0"/>
-      <geometry>
-        <box size="0.242 0.11 0.085"/>
-      </geometry>
-    </collision>
-</link>
-<link name="Inertia">
-<!-- !!!!!!!!!!!!!!!!!!!-->
-<!--NASTAVAIT SPRAVNE INERTIAL-->
-    <inertial>
-      <origin xyz="0 0 0.02" />
-      <mass value="1.172" />
-<!--	<mass value="1" />-->
-      <inertia  ixx="0.001568" ixy="0.0"  ixz="0.0"  iyy="0.003775"  iyz="0.0"  izz="0.00483" />
-    </inertial>
-</link>
-<joint name="$(arg prefix)base_link" type="fixed">
-	<parent link="$(arg prefix)base_link"/>
-	<child link="Inertia"/>
-	<origin xyz="0.0 0.0 0.0"/>
-</joint>
-<gazebo reference="$(arg prefix)base_link">
-	<material>Gazebo/GreyGradientSky</material>
-      <turnGravityOff>false</turnGravityOff>
- </gazebo>
-		<!-- *************** -->
-		<!-- Robots Elements -->
-		<!-- *************** -->
-		<!-- Here we create the robot elements using the xacro:macros imported at the beggining of this file -->
+	<xacro:property name="PI" value="3.1415926535897931"/>
+	<material name="gray_color">
+		<color rgba=".75 .75 .75 1"/>
+	</material>
+	<!-- LINKS -->
+	<!-- ////////////////////////////////////////////////// -->
+	<link name="$(arg prefix)base_link">
+		<visual>
+			<origin xyz="0.011 -0.060276 0" rpy="${PI/2} 0 ${PI/2}"/>
+			<geometry>
+				<mesh filename="package://mech_ros/robot_description/meshes/Chassis_10000.stl" scale="${Scale}"/>
+			</geometry>
+			<material name="gray_color"/>
+		</visual>
+		<collision>
+			<origin xyz="0.008 0 0.023" rpy="0 0 0"/>
+			<geometry>
+				<box size="0.242 0.11 0.085"/>
+			</geometry>
+		</collision>
+	</link>
+	<link name="Inertia">
+		<!-- !!!!!!!!!!!!!!!!!!!-->
+		<!--NASTAVAIT SPRAVNE INERTIAL-->
+		<inertial>
+			<origin xyz="0 0 0.02" />
+			<mass value="1.172" />
+			<!--	<mass value="1" />-->
+			<inertia ixx="0.001568" ixy="0.0" ixz="0.0" iyy="0.003775" iyz="0.0" izz="0.00483" />
+		</inertial>
+	</link>
+	<joint name="$(arg prefix)base_link" type="fixed">
+		<parent link="$(arg prefix)base_link"/>
+		<child link="Inertia"/>
+		<origin xyz="0.0 0.0 0.0"/>
+	</joint>
+	<gazebo reference="$(arg prefix)base_link">
+		<material>Gazebo/GreyGradientSky</material>
+		<turnGravityOff>false</turnGravityOff>
+	</gazebo>
+	<!-- *************** -->
+	<!-- Robots Elements -->
+	<!-- *************** -->
+	<!-- Here we create the robot elements using the xacro:macros imported at the beggining of this file -->
 	<xacro:rubber_wheel prefix="front_right" parent="$(arg prefix)base_link" reflect="false">
 		<origin xyz="${wheel_offset_x} -${wheel_offset_y} ${wheel_offset_z}" rpy="0 0 0"/>
@@ -99,17 +101,17 @@
 		<origin xyz="-${wheel_offset_x} -${wheel_offset_y} ${wheel_offset_z}" rpy="0 0 0"/>
 	</xacro:rubber_wheel>
-<!-- Import IMU -->
+	<!-- Import IMU -->
 	<xacro:sensor_imu_hector prefix="imu" parent="$(arg prefix)base_link">
 		<origin xyz="0 0.0 0.055" rpy="0 0 0"/>
 	</xacro:sensor_imu_hector>
-<!-- Import PiCamera -->
+	<!-- Import PiCamera -->
 	<xacro:pi_camera_sensor prefix="front" parent="$(arg prefix)base_link">
-<!--		<origin xyz="0.088 0 0.0204" rpy="0 0 0"/>-->
-	<origin xyz="0.088 0 0.0204" rpy="0 0 0"/>
+		<!--		<origin xyz="0.088 0 0.0204" rpy="0 0 0"/>-->
+		<origin xyz="0.088 0 0.0204" rpy="0 0 0"/>
 	</xacro:pi_camera_sensor>
-<!-- Import Laser -->
-	 <xacro:sensor_hokuyo_urg04lx prefix="laser" parent="$(arg prefix)base_link">
+	<!-- Import Laser -->
+	<xacro:sensor_hokuyo_urg04lx prefix="laser" parent="$(arg prefix)base_link">
 		<origin xyz="0.0 0.0 0.0804" rpy="0 0 0"/>
 	</xacro:sensor_hokuyo_urg04lx>
-<xacro:ros_control/>
+	<xacro:ros_control/>
 </robot>

File: robot_description/urdf/rubber_wheel.urdf.xacro (robot description, xacro)
@@ -29,5 +29,5 @@
 <xacro:property name="Scale" value="${scale} ${scale} ${scale}"/>
 <material name="tire_texture">
-    <texture filename="$(find mech_ros)/robot_description/textures/rubber.jpg" />
+    <texture filename="package://mech_ros/robot_description/textures/rubber.jpg" />
 </material>
   <xacro:macro name="rubber_wheel" params="prefix parent *origin reflect">
@@ -50,5 +50,5 @@
 	      </xacro:unless>
         <geometry>
-             <mesh filename="$(find mech_ros)/robot_description/meshes/Wheel_hub_simplified.stl" scale="${Scale}"/>
+             <mesh filename="package://mech_ros/robot_description/meshes/Wheel_hub_simplified.stl" scale="${Scale}"/>
         </geometry>
 	      <material name="tire_texture"/>
