Commit message: Add set pose to Kalman after docking, modified parameters from experiments

File: robot_description/urdf/rubber_wheel.urdf.xacro (robot description, xacro)
@@ -1,5 +1,6 @@
 <?xml version="1.0"?>
-<robot name="wheel" xmlns:xacro="http://www.ros.org/wiki/xacro">
-<!-- Copyright (c) 2014, Robotnik Automation
+<robot name="wheel"
+  xmlns:xacro="http://www.ros.org/wiki/xacro">
+  <!-- Copyright (c) 2014, Robotnik Automation
 All rights reserved.
 Redistribution and use in source and binary forms, with or without
@@ -23,14 +24,17 @@
   <!-- Wheels -->
   <xacro:property name="wheel_radius" value="0.05" />
-  <xacro:property name="wheel_height" value="0.031" /> <!-- really is the wheel width -->
-  <xacro:property name="wheel_mass" value="0.079" /> <!-- in kg-->
- <!-- SCALE definition -->
-<xacro:property name="scale" value="0.01"/>    <!-- meritko-->
-<xacro:property name="Scale" value="${scale} ${scale} ${scale}"/>
-<material name="tire_texture">
+  <xacro:property name="wheel_height" value="0.031" />
+  <!-- really is the wheel width -->
+  <xacro:property name="wheel_mass" value="0.079" />
+  <!-- in kg-->
+  <!-- SCALE definition -->
+  <xacro:property name="scale" value="0.01"/>
+  <!-- meritko-->
+  <xacro:property name="Scale" value="${scale} ${scale} ${scale}"/>
+  <material name="tire_texture">
     <texture filename="package://mech_ros/robot_description/textures/rubber.jpg" />
-</material>
+  </material>
   <xacro:macro name="rubber_wheel" params="prefix parent *origin reflect">
-<!--WHEEL TIRE -->
+    <!--WHEEL TIRE -->
     <joint name="${prefix}_wheel_joint" type="continuous">
       <parent link="${parent}"/>
@@ -43,22 +47,22 @@
     <link name="${prefix}_wheel">
       <visual>
-          <xacro:if value="${reflect}">
-		        <origin xyz="0 0.003 0" rpy="${-M_PI/2} 0 0" />
-	        </xacro:if>
-	      <xacro:unless value="${reflect}">
-		      <origin xyz="0 -0.003 0" rpy="${M_PI/2} 0 0" />
-	      </xacro:unless>
+        <xacro:if value="${reflect}">
+          <origin xyz="0 0.003 0" rpy="${-M_PI/2} 0 0" />
+        </xacro:if>
+        <xacro:unless value="${reflect}">
+          <origin xyz="0 -0.003 0" rpy="${M_PI/2} 0 0" />
+        </xacro:unless>
         <geometry>
-             <mesh filename="package://mech_ros/robot_description/meshes/Wheel_hub_simplified.stl" scale="${Scale}"/>
+          <mesh filename="package://mech_ros/robot_description/meshes/Wheel_hub_simplified.stl" scale="${Scale}"/>
         </geometry>
-	      <material name="tire_texture"/>
+        <material name="tire_texture"/>
       </visual>
       <collision>
-          <xacro:if value="${reflect}">
-		        <origin xyz="0 0.003 0" rpy="${M_PI/2} 0 0" />
-	        </xacro:if>
-	        <xacro:unless value="${reflect}">
-		        <origin xyz="0 -0.003 0" rpy="${M_PI/2} 0 0" />
-	        </xacro:unless>
+        <xacro:if value="${reflect}">
+          <origin xyz="0 0.003 0" rpy="${M_PI/2} 0 0" />
+        </xacro:if>
+        <xacro:unless value="${reflect}">
+          <origin xyz="0 -0.003 0" rpy="${M_PI/2} 0 0" />
+        </xacro:unless>
         <geometry>
           <cylinder length="${wheel_height}" radius="${wheel_radius}" />
@@ -78,18 +82,16 @@
       <inertial>
         <mass value="${wheel_mass}" />
-	      <xacro:if value="${reflect}">
-		      <origin xyz="0 0.003 0" rpy="0 0 0" />
-	      </xacro:if>
-	      <xacro:unless value="${reflect}">
-		      <origin xyz="0 -0.003 0" rpy="0 0 0" />
-	      </xacro:unless>
+        <xacro:if value="${reflect}">
+          <origin xyz="0 0.003 0" rpy="0 0 0" />
+        </xacro:if>
+        <xacro:unless value="${reflect}">
+          <origin xyz="0 -0.003 0" rpy="0 0 0" />
+        </xacro:unless>
         <!-- <origin xyz="0 0 0" /> -->
-	      <inertia  ixx="0.00069" ixy = "0" ixz = "0"
-              iyy="0.0012057" iyz = "0"
-              izz="0.00069" />
-        </inertial>
+        <inertia ixx="0.00069" ixy = "0" ixz = "0" iyy="0.0012057" iyz = "0" izz="0.00069" />
+      </inertial>
     </link>
     <!-- Transmission is important to link the joints and the controller (see summit_xl_control/config/summit_xl_control.yaml)-->
-	<transmission name="${prefix}_wheel_joint_trans">
+    <transmission name="${prefix}_wheel_joint_trans">
       <type>transmission_interface/SimpleTransmission</type>
       <joint name="${prefix}_wheel_joint">
@@ -103,5 +105,5 @@
     </transmission>
     <gazebo reference="${prefix}_wheel">
-	    <material>Gazebo/Residential</material>
+      <material>Gazebo/Residential</material>
       <turnGravityOff>false</turnGravityOff>
     </gazebo>
